Commit message: update
now the rviz is working.
**bug** for some reason, the image of the robot is not being displayed on rviz. @pchavez201706
if you find any syntax errors pls lmk..

File: ros2/ros2-pkg/hos-resolve/src/mycobot_description/urdf/mycobot_320_pi_2022/mycobot_320_pi_moveit_2022_gz.urdf (robot description, URDF)
Before this commit: robot firefighter, 7 links, 6 joints
Links:
- link base: geometry collision cylinder length=0.102 radius=0.0725; visual mesh filename=file://$(find mycobot_description)/urdf/mycobot_320_pi_2022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
- link link1: geometry collision cylinder length=0.106 radius=0.043; visual mesh filename=file://$(find mycobot_description)/urdf/mycobot_320_pi_2022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
- link link2: geometry collision cylinder length=0.18 radius=0.036; visual mesh filename=file://$(find mycobot_description)/urdf/mycobot_320_pi_2022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
- link link3: geometry collision cylinder length=0.14 radius=0.0305; visual mesh filename=file://$(find mycobot_description)/urdf/mycobot_320_pi_2022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
- link link4: geometry collision cylinder length=0.083 radius=0.029; visual mesh filename=file://$(find mycobot_description)/urdf/mycobot_320_pi_2022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
- link link5: geometry collision cylinder length=0.0849 radius=0.029; visual mesh filename=file://$(find mycobot_description)/urdf/mycobot_320_pi_2022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
- link link6: geometry collision cylinder length=0.0225 radius=0.026; visual mesh filename=file://$(find mycobot_description)/urdf/mycobot_320_pi_2022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

File: ros2/ros2-pkg/hos-resolve/src/mycobot_description/urdf/mycobot_320_pi_2022/mycobot_320_pi_moveit_2022_gz.urdf.xacro (robot description, xacro)
@@ -1,30 +1,7 @@
 <?xml version="1.0" ?>
-<robot xmlns:xacro="http://wiki.ros.org/xacro" name="mycobot_320pi">
-	<!--
-		xml:
-			Declare this file as an XML document and specifies the XML version.
-		robot:
-			The root element 'robot' defines a robot model. Everything about the
-			robot configuration will be nested inside this element.
-		xmlns:xacro:
-			Declares the XML namespace for xacro, which is a XML macro language used
-			in ROS (Robot Operating System) for parameterizing XML documents.
-		name:
-			Specify the name of the robot.
-	-->
-	<!-- Reference Files: https://github.com/elephantrobotics/mycobot_ros/ -->
-	<!-- Provide a global reference frame for the robotic arm in simulation (Gazebo)
-		or visualization (RViz) environments
-	-->
+<robot xmlns:xacro="http://wiki.ros.org/xacro" name="mycobot_280">
 	<link name="world"/>
-	<!-- ****************** ROBOT CONSTANTS *******************************  -->
-	<!-- Source: https://www.elephantrobotics.com/en/mycobot280-for-arduino-specifications-en/ -->
-	<!-- Numbers are estimated when necessary -->
-	<xacro:property name="effort" value="5.0"/> <!-- TODO: effort is 1000.00?? -->
+	<xacro:property name="effort" value="5.0"/> <!-- WHAT: effort is 1000.00?? -->
 	<xacro:property name="velocity" value="2.792527"/>
-	<!-- ********** LINKS ********** -->
-    <!-- Define the base plate of the robotic arm
-    	The inertial values below were taken from link1 (with slight modification.
-		They are just placeholder values. -->
 	<link name="base">
 		<inertial>
@@ -38,16 +15,15 @@
 		<visual>
 			<geometry>
-				<mesh filename="/home/cfh/Desktop/ClawForHumanity/hos-resolve/install/mycobot_description/share/mycobot_description/urdf/mycobot_320_pi_2022/base.dae"/>
-			</geometry>
-			<origin xyz = "0.0 0 0 " rpy = " 0 0 1.5708"/>
-		</visual>
-		<collision>
-			<origin xyz = "0.0 0 0 " rpy = " 0 0 1.5708"/>
-			<geometry>
-				<cylinder length="0.102" radius="0.0725"/>
-			</geometry>
-		</collision>
-	</link>
-	<!--Define the first link of the robotic arm. Each link represents a solid part of the robot.-->
+				<mesh filename="file://$(find mycobot_description)/urdf/mycobot_320_pi_2022/base.dae"/>
+			</geometry>
+			<origin xyz = "0.0 0 0 " rpy = "0 0 ${pi/2}"/>
+		</visual>
+		<collision>
+			<geometry>
+				<mesh filename="file://$(find mycobot_description)/urdf/mycobot_320_pi_2022/base.dae"/>
+			</geometry>
+			<origin xyz = "0.0 0 0 " rpy = "0 0 ${pi/2}"/>
+		</collision>
+	</link>
 	<link name="link1">
 		<inertial>
@@ -61,16 +37,15 @@
 		<visual>
 			<geometry>
-				<mesh filename="/home/cfh/Desktop/ClawForHumanity/hos-resolve/install/mycobot_description/share/mycobot_description/urdf/mycobot_320_pi_2022/link1.dae"/>
-			</geometry>
-			<origin xyz = "0.0 0.0 -0.078 " rpy = " 0 0 1.5708"/>
-		</visual>
-		<collision>
-			<origin xyz = "0.0 0.0 -0.078 " rpy = " 0 0 1.5708"/>
-			<geometry>
-				<cylinder length="0.106" radius="0.043"/>
-			</geometry>
-		</collision>
-	</link>
-	<!-- Define the second link of the robotic arm, and so on.-->
+				<mesh filename="file://$(find mycobot_description)/urdf/mycobot_320_pi_2022/link1.dae"/>
+			</geometry>
+			<origin xyz = "0.0 0 -0.078 " rpy = " 0 0 ${pi/2}"/>
+		</visual>
+		<collision>
+			<geometry>
+				<mesh filename="file://$(find mycobot_description)/urdf/mycobot_320_pi_2022/link1.dae"/>
+			</geometry>
+			<origin xyz = "0.0 0 -0.078 " rpy = " 0 0 ${pi/2}"/>
+		</collision>
+	</link>
 	<link name="link2">
 		<inertial>
@@ -84,13 +59,13 @@
 		<visual>
 			<geometry>
-				<mesh filename="/home/cfh/Desktop/ClawForHumanity/hos-resolve/install/mycobot_description/share/mycobot_description/urdf/mycobot_320_pi_2022/link2.dae"/>
-			</geometry>
-			<origin xyz = "0.0 0.0 -0.04 " rpy = " 0 1.5708 0"/>
-		</visual>
-		<collision>
-			<origin xyz = "0.0 0.0 -0.04 " rpy = " 0 1.5708 0"/>
-			<geometry>
-				<cylinder length="0.18" radius="0.036"/>
-			</geometry>
+				<mesh filename="file://$(find mycobot_description)/urdf/mycobot_320_pi_2022/link2.dae"/>
+			</geometry>
+			<origin xyz = "0.0 0 -0.04 " rpy = " 0 ${pi/2} 0"/>
+		</visual>
+		<collision>
+			<geometry>
+				<mesh filename="file://$(find mycobot_description)/urdf/mycobot_320_pi_2022/link2.dae"/>
+			</geometry>
+			<origin xyz = "0.0 0 -0.04 " rpy = " 0 ${pi/2} 0"/>
 		</collision>
 	</link>
@@ -105,15 +80,15 @@
 		</inertial>
 		<visual>
-      		<geometry>
-        		<mesh filename="/home/cfh/Desktop/ClawForHumanity/hos-resolve/install/mycobot_description/share/mycobot_description/urdf/mycobot_320_pi_2022/link3.dae"/>
-      		</geometry>
-     		<origin xyz = "0.0 0.0 0.039 " rpy = " 1.5708 1.5708 1.5708"/>
-    	</visual>
-    	<collision>
-      		<origin xyz = "0.0 0.0 0.039 " rpy = " 1.5708 1.5708 1.5708"/>
-      		<geometry>
-        		<cylinder length="0.14" radius="0.0305"/>
-      		</geometry>
-    	</collision>
+		  	<geometry>
+		   		<mesh filename="file://$(find mycobot_description)/urdf/mycobot_320_pi_2022/link3.dae"/>
+		  	</geometry>
+			<origin xyz = "0.0 0 0.039 " rpy = " ${pi/2} ${pi/2} ${pi/2}"/>
+		</visual>
+		<collision>
+		  	<geometry>
+		   		<mesh filename="file://$(find mycobot_description)/urdf/mycobot_320_pi_2022/link3.dae"/>
+		  	</geometry>
+		  	<origin xyz = "0.0 0 0.039 " rpy = " ${pi/2} ${pi/2} ${pi/2}"/>
+		</collision>
 	</link>
 	<link name="link4">
@@ -128,13 +103,13 @@
 		<visual>
 			<geometry>
-				<mesh filename="/home/cfh/Desktop/ClawForHumanity/hos-resolve/install/mycobot_description/share/mycobot_description/urdf/mycobot_320_pi_2022/link4.dae"/>
-			</geometry>
-			<origin xyz = "0.0 -0.0024 -0.05" rpy = " 1.5708 1.5708 0"/>
-		</visual>
-		<collision>
-			<origin xyz = "0.0 -0.0024 -0.05" rpy = " 1.5708 1.5708 0"/>
-			<geometry>
-				<cylinder length="0.083" radius="0.029"/>
-			</geometry>
+				<mesh filename="file://$(find mycobot_description)/urdf/mycobot_320_pi_2022/link4.dae"/>
+			</geometry>
+			<origin xyz = "0.0 -0.0024 -0.05 " rpy = "${pi/2} ${pi/2} 0 "/>
+		</visual>
+		<collision>
+			<geometry>
+				<mesh filename="file://$(find mycobot_description)/urdf/mycobot_320_pi_2022/link4.dae"/>
+			</geometry>
+			<origin xyz = "0.0 -0.0024 -0.05 " rpy = "${pi/2} ${pi/2} 0 "/>
 		</collision>
 	</link>
@@ -149,14 +124,14 @@
 		</inertial>
 		<visual>
-			<geometry>
-				<mesh filename="/home/cfh/Desktop/ClawForHumanity/hos-resolve/install/mycobot_description/share/mycobot_description/urdf/mycobot_320_pi_2022/link5.dae"/>
-			</geometry>
-			<origin xyz = "0.0 0.0 -0.05 " rpy = " 0  0 -1.5708"/>
-		</visual>
-		<collision>
-			<origin xyz = "0.0 0.0 -0.05 " rpy = " 0  0 -1.5708"/>
-			<geometry>
-				<cylinder length="0.0849" radius="0.029"/>
-			</geometry>
+		  	<geometry>
+				<mesh filename="file://$(find mycobot_description)/urdf/mycobot_320_pi_2022/link5.dae"/>
+		  	</geometry>
+		  	<origin xyz = "0.0 0 -0.05 " rpy = "0 0 ${-pi/2}"/>
+		</visual>
+		<collision>
+		   	<geometry>
+		   		<mesh filename="file://$(find mycobot_description)/urdf/mycobot_320_pi_2022/link5.dae"/>
+		  	</geometry>
+		  	<origin xyz = "0.0 0 -0.05 " rpy = "0 0 ${-pi/2}"/>
 		</collision>
 	</link>
@@ -172,42 +147,18 @@
 		<visual>
 			<geometry>
-				<mesh filename="/home/cfh/Desktop/ClawForHumanity/hos-resolve/install/mycobot_description/share/mycobot_description/urdf/mycobot_320_pi_2022/link6.dae"/>
+				<mesh filename="file://$(find mycobot_description)/urdf/mycobot_320_pi_2022/link6.dae"/>
 			</geometry>
 			<material name = "grey">
 				<color rgba = "0.5 0.5 0.5 1"/>
 			</material>
-				<origin xyz = "0.0 0.0 -0.022 " rpy = " 1.5708 1.5708 0"/>
-		</visual>
-		<collision>
-			<origin xyz = "0.0 0.0 -0.022 " rpy = " 1.5708 1.5708 0"/>
-			<geometry>
-				<cylinder length="0.0225" radius="0.026"/>
-		</geometry>
-		</collision>
-	</link>
-    <!-- ********** COLORS ********** -->
-    <gazebo reference="base">
-        <material>Gazebo/Grey</material>
-    </gazebo>
-    <gazebo reference="link1">
-        <material>Gazebo/White</material>
-    </gazebo>
-    <gazebo reference="link2">
-        <material>Gazebo/White</material>
-    </gazebo>
-    <gazebo reference="link3">
-        <material>Gazebo/White</material>
-    </gazebo>
-    <gazebo reference="link4">
-        <material>Gazebo/White</material>
-    </gazebo>
-    <gazebo reference="link5">
-        <material>Gazebo/White</material>
-    </gazebo>
-    <gazebo reference="link6">
-        <material>Gazebo/White</material>
-    </gazebo>
-	<!-- ********** JOINTS ********** -->
-	<!-- Attach the robot base to the world frame with no initial offset or rotation. -->
+				<origin xyz = "0.0 0.0 -0.022 " rpy = " ${pi/2} ${pi/2} 0"/>
+		</visual>
+		<collision>
+		   	<geometry>
+		   		<mesh filename="file://$(find mycobot_description)/urdf/mycobot_320_pi_2022/link6.dae"/>
+		  	</geometry>
+		  	<origin xyz = "0.0 0.0 -0.022 " rpy = " ${pi/2} ${pi/2} 0"/>
+		</collision>
+	</link>
 	<joint name="virtual_joint" type="fixed">
 		<parent link="world"/>
@@ -263,29 +214,38 @@
         <dynamics damping="3.0" friction="3.0"/>
 	</joint>
-	<!-- The mimic element means this joint will follow the movements of the
-		gripper_controller joint.
-	-->
-	<!-- ********** PLUGINS ********** -->
-    <!-- Publishes joint state information for the model which the robot_state_publisher uses to broadcast to
-            the tf topic, the topic that keeps track of the robot's multiple coordinate frames over time -->
-    <gazebo>
-        <plugin name="gazebo_ros_joint_state_publisher" filename="libgazebo_ros_joint_state_publisher.so">
-            <update_rate>20</update_rate>
+    <gazebo>
+        <plugin filename="ignition-gazebo-joint-state-publisher-system" name="ignition::gazebo::systems::JointStatePublisher">
+            <topic>joint_states</topic>
+        </plugin>
+    </gazebo>
+    <gazebo>
+        <plugin filename="ignition-gazebo-joint-position-controller-system" name="ignition::gazebo::systems::JointPositionController">
             <joint_name>joint2_to_joint1</joint_name>
+        </plugin>
+    </gazebo>
+    <gazebo>
+        <plugin filename="ignition-gazebo-joint-position-controller-system" name="ignition::gazebo::systems::JointPositionController">
             <joint_name>joint3_to_joint2</joint_name>
+        </plugin>
+    </gazebo>
+    <gazebo>
+        <plugin filename="ignition-gazebo-joint-position-controller-system" name="ignition::gazebo::systems::JointPositionController">
             <joint_name>joint4_to_joint3</joint_name>
+        </plugin>
+    </gazebo>
+    <gazebo>
+        <plugin filename="ignition-gazebo-joint-position-controller-system" name="ignition::gazebo::systems::JointPositionController">
             <joint_name>joint5_to_joint4</joint_name>
+        </plugin>
+    </gazebo>
+    <gazebo>
+        <plugin filename="ignition-gazebo-joint-position-controller-system" name="ignition::gazebo::systems::JointPositionController">
             <joint_name>joint6_to_joint5</joint_name>
+        </plugin>
+    </gazebo>
+    <gazebo>
+        <plugin filename="ignition-gazebo-joint-position-controller-system" name="ignition::gazebo::systems::JointPositionController">
             <joint_name>joint6output_to_joint6</joint_name>
         </plugin>
     </gazebo>
-    <!-- Subscribes to a JointTrajectory message from the /set_joint_trajectory topic
-        To publish to this topic type:
-            ros2 topic pub -1 /set_joint_trajectory trajectory_msgs/msg/JointTrajectory "{header: {frame_id: base_link}, joint_names: [link1_to_link2, link2_to_link3, etc.], points: [{positions: [0.0,0.0,etc.]}]}"
-    -->
-    <gazebo>
-        <plugin name="gazebo_ros_joint_pose_trajectory" filename="libgazebo_ros_joint_pose_trajectory.so">
-            <update_rate>20</update_rate>
-        </plugin>
-    </gazebo>
 </robot>
