Commit message: organize & restructure
organised codes and folders.
Now the package is renamed to mycobot_320pi_gz

File: ros2/ros2-pkg/hos-resolve/src/mycobot_320pi_gz/config/firefighter.urdf.xacro (robot description, xacro)
@@ -3,5 +3,5 @@
     <xacro:arg name="initial_positions_file" default="initial_positions.yaml" />
     <!-- Import firefighter urdf file -->
-    <xacro:include filename="$(find mycobot_description)/urdf/mycobot_320_pi_2022/mycobot_320_pi_moveit_2022.urdf" />
+    <xacro:include filename="$(find mycobot_description)/urdf/original/mycobot_320_pi_moveit_2022.urdf" />
     <!-- Import control_xacro -->
     <xacro:include filename="firefighter.ros2_control.xacro" />

File: ros2/ros2-pkg/hos-resolve/src/mycobot_description/urdf/xacro/mycobot_320_pi_gz.urdf.xacro (robot description, xacro)
@@ -15,5 +15,5 @@
 		<visual>
 			<geometry>
-				<mesh filename="file://$(find mycobot_description)/urdf/mycobot_320_pi_2022/base.dae"/>
+				<mesh filename="file://$(find mycobot_description)/urdf/mesh/base.dae"/>
 			</geometry>
 			<origin xyz = "0.0 0 0 " rpy = "0 0 ${pi/2}"/>
@@ -21,5 +21,5 @@
 		<collision>
 			<geometry>
-				<mesh filename="file://$(find mycobot_description)/urdf/mycobot_320_pi_2022/base.dae"/>
+				<mesh filename="file://$(find mycobot_description)/urdf/mesh/base.dae"/>
 			</geometry>
 			<origin xyz = "0.0 0 0 " rpy = "0 0 ${pi/2}"/>
@@ -37,5 +37,5 @@
 		<visual>
 			<geometry>
-				<mesh filename="file://$(find mycobot_description)/urdf/mycobot_320_pi_2022/link1.dae"/>
+				<mesh filename="file://$(find mycobot_description)/urdf/mesh/link1.dae"/>
 			</geometry>
 			<origin xyz = "0.0 0 -0.078 " rpy = " 0 0 ${pi/2}"/>
@@ -43,5 +43,5 @@
 		<collision>
 			<geometry>
-				<mesh filename="file://$(find mycobot_description)/urdf/mycobot_320_pi_2022/link1.dae"/>
+				<mesh filename="file://$(find mycobot_description)/urdf/mesh/link1.dae"/>
 			</geometry>
 			<origin xyz = "0.0 0 -0.078 " rpy = " 0 0 ${pi/2}"/>
@@ -59,5 +59,5 @@
 		<visual>
 			<geometry>
-				<mesh filename="file://$(find mycobot_description)/urdf/mycobot_320_pi_2022/link2.dae"/>
+				<mesh filename="file://$(find mycobot_description)/urdf/mesh/link2.dae"/>
 			</geometry>
 			<origin xyz = "0.0 0 -0.04 " rpy = " 0 ${pi/2} 0"/>
@@ -65,5 +65,5 @@
 		<collision>
 			<geometry>
-				<mesh filename="file://$(find mycobot_description)/urdf/mycobot_320_pi_2022/link2.dae"/>
+				<mesh filename="file://$(find mycobot_description)/urdf/mesh/link2.dae"/>
 			</geometry>
 			<origin xyz = "0.0 0 -0.04 " rpy = " 0 ${pi/2} 0"/>
@@ -81,5 +81,5 @@
 		<visual>
 		  	<geometry>
-		   		<mesh filename="file://$(find mycobot_description)/urdf/mycobot_320_pi_2022/link3.dae"/>
+		   		<mesh filename="file://$(find mycobot_description)/urdf/mesh/link3.dae"/>
 		  	</geometry>
 			<origin xyz = "0.0 0 0.039 " rpy = " ${pi/2} ${pi/2} ${pi/2}"/>
@@ -87,5 +87,5 @@
 		<collision>
 		  	<geometry>
-		   		<mesh filename="file://$(find mycobot_description)/urdf/mycobot_320_pi_2022/link3.dae"/>
+		   		<mesh filename="file://$(find mycobot_description)/urdf/mesh/link3.dae"/>
 		  	</geometry>
 		  	<origin xyz = "0.0 0 0.039 " rpy = " ${pi/2} ${pi/2} ${pi/2}"/>
@@ -103,5 +103,5 @@
 		<visual>
 			<geometry>
-				<mesh filename="file://$(find mycobot_description)/urdf/mycobot_320_pi_2022/link4.dae"/>
+				<mesh filename="file://$(find mycobot_description)/urdf/mesh/link4.dae"/>
 			</geometry>
 			<origin xyz = "0.0 -0.0024 -0.05 " rpy = "${pi/2} ${pi/2} 0 "/>
@@ -109,5 +109,5 @@
 		<collision>
 			<geometry>
-				<mesh filename="file://$(find mycobot_description)/urdf/mycobot_320_pi_2022/link4.dae"/>
+				<mesh filename="file://$(find mycobot_description)/urdf/mesh/link4.dae"/>
 			</geometry>
 			<origin xyz = "0.0 -0.0024 -0.05 " rpy = "${pi/2} ${pi/2} 0 "/>
@@ -125,5 +125,5 @@
 		<visual>
 		  	<geometry>
-				<mesh filename="file://$(find mycobot_description)/urdf/mycobot_320_pi_2022/link5.dae"/>
+				<mesh filename="file://$(find mycobot_description)/urdf/mesh/link5.dae"/>
 		  	</geometry>
 		  	<origin xyz = "0.0 0 -0.05 " rpy = "0 0 ${-pi/2}"/>
@@ -131,5 +131,5 @@
 		<collision>
 		   	<geometry>
-		   		<mesh filename="file://$(find mycobot_description)/urdf/mycobot_320_pi_2022/link5.dae"/>
+		   		<mesh filename="file://$(find mycobot_description)/urdf/mesh/link5.dae"/>
 		  	</geometry>
 		  	<origin xyz = "0.0 0 -0.05 " rpy = "0 0 ${-pi/2}"/>
@@ -147,5 +147,5 @@
 		<visual>
 			<geometry>
-				<mesh filename="file://$(find mycobot_description)/urdf/mycobot_320_pi_2022/link6.dae"/>
+				<mesh filename="file://$(find mycobot_description)/urdf/mesh/link6.dae"/>
 			</geometry>
 			<material name = "grey">
@@ -156,5 +156,5 @@
 		<collision>
 		   	<geometry>
-		   		<mesh filename="file://$(find mycobot_description)/urdf/mycobot_320_pi_2022/link6.dae"/>
+		   		<mesh filename="file://$(find mycobot_description)/urdf/mesh/link6.dae"/>
 		  	</geometry>
 		  	<origin xyz = "0.0 0.0 -0.022 " rpy = " ${pi/2} ${pi/2} 0"/>

File: ros2/ros2-pkg/hos-resolve/src/mycobot_description/urdf/xacro/mycobot_320_pi_ros2control.urdf.xacro (robot description, xacro)
@@ -1,30 +1,7 @@
 <?xml version="1.0" ?>
 <robot xmlns:xacro="http://wiki.ros.org/xacro" name="mycobot_320pi">
-	<!--
-		xml:
-			Declare this file as an XML document and specifies the XML version.
-		robot:
-			The root element 'robot' defines a robot model. Everything about the
-			robot configuration will be nested inside this element.
-		xmlns:xacro:
-			Declares the XML namespace for xacro, which is a XML macro language used
-			in ROS (Robot Operating System) for parameterizing XML documents.
-		name:
-			Specify the name of the robot.
-	-->
-	<!-- Reference Files: https://github.com/elephantrobotics/mycobot_ros/ -->
-	<!-- Provide a global reference frame for the robotic arm in simulation (Gazebo)
-		or visualization (RViz) environments
-	-->
 	<link name="world"/>
-	<!-- ****************** ROBOT CONSTANTS *******************************  -->
-	<!-- Source: https://www.elephantrobotics.com/en/mycobot280-for-arduino-specifications-en/ -->
-	<!-- Numbers are estimated when necessary -->
 	<xacro:property name="effort" value="5.0"/> <!-- TODO: effort is 1000.00?? -->
 	<xacro:property name="velocity" value="2.792527"/>
-	<!-- ********** LINKS ********** -->
-    <!-- Define the base plate of the robotic arm
-    	The inertial values below were taken from link1 (with slight modification.
-		They are just placeholder values. -->
 	<link name="base">
 		<inertial>
@@ -38,5 +15,5 @@
 		<visual>
 			<geometry>
-				<mesh filename="file://$(find mycobot_description)/urdf/mycobot_320_pi_2022/base.dae"/>
+				<mesh filename="file://$(find mycobot_description)/urdf/mesh/base.dae"/>
 			</geometry>
 			<origin xyz = "0.0 0 0 " rpy = " 0 0 1.5708"/>
@@ -61,5 +38,5 @@
 		<visual>
 			<geometry>
-				<mesh filename="file://$(find mycobot_description)/urdf/mycobot_320_pi_2022/link1.dae"/>
+				<mesh filename="file://$(find mycobot_description)/urdf/mesh/link1.dae"/>
 			</geometry>
 			<origin xyz = "0.0 0.0 -0.078 " rpy = " 0 0 1.5708"/>
@@ -84,5 +61,5 @@
 		<visual>
 			<geometry>
-				<mesh filename="file://$(find mycobot_description)/urdf/mycobot_320_pi_2022/link2.dae"/>
+				<mesh filename="file://$(find mycobot_description)/urdf/mesh/link2.dae"/>
 			</geometry>
 			<origin xyz = "0.0 0 -0.04 " rpy = " 0 1.5708 0"/>
@@ -106,5 +83,5 @@
 		<visual>
       		<geometry>
-        		<mesh filename="file://$(find mycobot_description)/urdf/mycobot_320_pi_2022/link3.dae"/>
+        		<mesh filename="file://$(find mycobot_description)/urdf/mesh/link3.dae"/>
       		</geometry>
      		<origin xyz = "0.0 0.0 0.039 " rpy = " 1.5708 1.5708 1.5708"/>
@@ -128,5 +105,5 @@
 		<visual>
 			<geometry>
-				<mesh filename="file://$(find mycobot_description)/urdf/mycobot_320_pi_2022/link4.dae"/>
+				<mesh filename="file://$(find mycobot_description)/urdf/mesh/link4.dae"/>
 			</geometry>
 			<origin xyz = "0.0 -0.0024 -0.05 " rpy = " 1.5708 1.5708 0"/>
@@ -150,5 +127,5 @@
 		<visual>
 			<geometry>
-				<mesh filename="file://$(find mycobot_description)/urdf/mycobot_320_pi_2022/link5.dae"/>
+				<mesh filename="file://$(find mycobot_description)/urdf/mesh/link5.dae"/>
 			</geometry>
 			<origin xyz = "0.0 0.0 -0.05 " rpy = " 0  0 -1.5708"/>
@@ -172,5 +149,5 @@
 		<visual>
 			<geometry>
-				<mesh filename="file://$(find mycobot_description)/urdf/mycobot_320_pi_2022/link6.dae"/>
+				<mesh filename="file://$(find mycobot_description)/urdf/mesh/link6.dae"/>
 			</geometry>
 			<material name = "grey">
@@ -263,10 +240,4 @@
         <dynamics damping="3.0" friction="3.0"/>
 	</joint>
-	<!-- The mimic element means this joint will follow the movements of the
-		gripper_controller joint.
-	-->
-	<!-- ********** PLUGINS ********** -->
-    <!-- Publishes joint state information for the model which the robot_state_publisher uses to broadcast to
-            the tf topic, the topic that keeps track of the robot's multiple coordinate frames over time -->
     <gazebo>
         <plugin name="gazebo_ros_joint_state_publisher" filename="libgazebo_ros_joint_state_publisher.so">
@@ -280,8 +251,4 @@
         </plugin>
     </gazebo>
-    <!-- Subscribes to a JointTrajectory message from the /set_joint_trajectory topic
-        To publish to this topic type:
-            ros2 topic pub -1 /set_joint_trajectory trajectory_msgs/msg/JointTrajectory "{header: {frame_id: base_link}, joint_names: [link1_to_link2, link2_to_link3, etc.], points: [{positions: [0.0,0.0,etc.]}]}"
-    -->
     <gazebo>
         <plugin name="gazebo_ros_joint_pose_trajectory" filename="libgazebo_ros_joint_pose_trajectory.so">
