Commit message: moveit2 wip

File: ros2/ros2-pkg/hos-resolve/src/mycobot_description/urdf/original/mycobot_320_pi_2022.urdf (robot description, URDF)
Before this commit: robot firefighter, 7 links, 6 joints
Links:
- link base: geometry collision mesh filename=package://mycobot_description/urdf/mesh/base.dae; visual mesh filename=package://mycobot_description/urdf/mesh/base.dae
- link link1: geometry collision mesh filename=package://mycobot_description/urdf/mesh/link1.dae; visual mesh filename=package://mycobot_description/urdf/mesh/link1.dae
- link link2: geometry collision mesh filename=package://mycobot_description/urdf/mesh/link2.dae; visual mesh filename=package://mycobot_description/urdf/mesh/link2.dae
- link link3: geometry collision mesh filename=package://mycobot_description/urdf/mesh/link3.dae; visual mesh filename=package://mycobot_description/urdf/mesh/link3.dae
- link link4: geometry collision mesh filename=package://mycobot_description/urdf/mesh/link4.dae; visual mesh filename=package://mycobot_description/urdf/mesh/link4.dae
- link link5: geometry collision mesh filename=package://mycobot_description/urdf/mesh/link5.dae; visual mesh filename=package://mycobot_description/urdf/mesh/link5.dae
- link link6: geometry collision mesh filename=package://mycobot_description/urdf/mesh/link6.dae; visual mesh filename=package://mycobot_description/urdf/mesh/link6.dae

File: ros2/ros2-pkg/hos-resolve/src/mycobot_description/urdf/original/mycobot_320_pi_moveit_2022.urdf (robot description, URDF)
Before this commit: robot firefighter, 7 links, 6 joints
Links:
- link base: geometry collision cylinder length=0.102 radius=0.0725; visual mesh filename=package://mycobot_description/urdf/mesh/base.dae
- link link1: geometry collision cylinder length=0.106 radius=0.043; visual mesh filename=package://mycobot_description/urdf/mesh/link1.dae
- link link2: geometry collision cylinder length=0.18 radius=0.036; visual mesh filename=package://mycobot_description/urdf/mesh/link2.dae
- link link3: geometry collision cylinder length=0.14 radius=0.0305; visual mesh filename=package://mycobot_description/urdf/mesh/link3.dae
- link link4: geometry collision cylinder length=0.083 radius=0.029; visual mesh filename=package://mycobot_description/urdf/mesh/link4.dae
- link link5: geometry collision cylinder length=0.0849 radius=0.029; visual mesh filename=package://mycobot_description/urdf/mesh/link5.dae
- link link6: geometry collision cylinder length=0.0225 radius=0.026; visual mesh filename=package://mycobot_description/urdf/mesh/link6.dae

File: ros2/ros2-pkg/hos-resolve/src/mycobot_description/urdf/original/mycobot_320_pi_moveit_2022_gz.urdf (robot description, URDF)
Before this commit: robot firefighter, 7 links, 6 joints
Links:
- link base: geometry collision cylinder length=0.102 radius=0.0725; visual mesh filename=file://$(find mycobot_description)/urdf/mesh/base.dae
- link link1: geometry collision cylinder length=0.106 radius=0.043; visual mesh filename=file://$(find mycobot_description)/urdf/mesh/link1.dae
- link link2: geometry collision cylinder length=0.18 radius=0.036; visual mesh filename=file://$(find mycobot_description)/urdf/mesh/link2.dae
- link link3: geometry collision cylinder length=0.14 radius=0.0305; visual mesh filename=file://$(find mycobot_description)/urdf/mesh/link3.dae
- link link4: geometry collision cylinder length=0.083 radius=0.029; visual mesh filename=file://$(find mycobot_description)/urdf/mesh/link4.dae
- link link5: geometry collision cylinder length=0.0849 radius=0.029; visual mesh filename=file://$(find mycobot_description)/urdf/mesh/link5.dae
- link link6: geometry collision cylinder length=0.0225 radius=0.026; visual mesh filename=file://$(find mycobot_description)/urdf/mesh/link6.dae

File: ros2/ros2-pkg/hos-resolve/src/mycobot_description/urdf/original/mycobot_vision_v2_2022.urdf (robot description, URDF)
Before this commit: robot firefighter, 8 links, 7 joints
Links:
- link base: geometry collision mesh filename=package://mycobot_description/urdf/mesh/base.dae; visual mesh filename=package://mycobot_description/urdf/mesh/base.dae
- link env: geometry visual mesh filename=package://mycobot_description/urdf/mesh/ai_kit320.dae
- link link1: geometry collision mesh filename=package://mycobot_description/urdf/mesh/link1.dae; visual mesh filename=package://mycobot_description/urdf/mesh/link1.dae
- link link2: geometry collision mesh filename=package://mycobot_description/urdf/mesh/link2.dae; visual mesh filename=package://mycobot_description/urdf/mesh/link2.dae
- link link3: geometry collision mesh filename=package://mycobot_description/urdf/mesh/link3.dae; visual mesh filename=package://mycobot_description/urdf/mesh/link3.dae
- link link4: geometry collision mesh filename=package://mycobot_description/urdf/mesh/link4.dae; visual mesh filename=package://mycobot_description/urdf/mesh/link4.dae
- link link5: geometry collision mesh filename=package://mycobot_description/urdf/mesh/link5.dae; visual mesh filename=package://mycobot_description/urdf/mesh/link5.dae
- link link6: geometry collision mesh filename=package://mycobot_description/urdf/mesh/link6.dae; visual mesh filename=package://mycobot_description/urdf/mesh/link6.dae
