Commit message: moveit2 integration wip
created new urdf that doesn't cause invalid initial position bug.
launch file modified for moveit2 integration.

File: ros2/ros2-pkg/hos-resolve/src/mycobot_description/urdf/xacro/mycobot_320_pi_gz.urdf_v2.xacro (robot description, xacro)
@@ -20,8 +20,8 @@
 		</visual>
 		<collision>
-			<geometry>
-				<mesh filename="file://$(find mycobot_description)/urdf/mesh/base.dae"/>
-			</geometry>
-			<origin xyz = "0.0 0 0 " rpy = "0 0 ${pi/2}"/>
+			<origin xyz = "0.0 0 0 " rpy = " 0 0 ${pi/2}"/>
+			<geometry>
+				<cylinder length="0.102" radius="0.0725"/>
+			</geometry>
 		</collision>
 	</link>
@@ -42,8 +42,8 @@
 		</visual>
 		<collision>
-			<geometry>
-				<mesh filename="file://$(find mycobot_description)/urdf/mesh/link1.dae"/>
-			</geometry>
 			<origin xyz = "0.0 0 -0.078 " rpy = " 0 0 ${pi/2}"/>
+			<geometry>
+				<cylinder length="0.106" radius="0.043"/>
+			</geometry>
 		</collision>
 	</link>
@@ -64,8 +64,8 @@
 		</visual>
 		<collision>
-			<geometry>
-				<mesh filename="file://$(find mycobot_description)/urdf/mesh/link2.dae"/>
-			</geometry>
 			<origin xyz = "0.0 0 -0.04 " rpy = " 0 ${pi/2} 0"/>
+			<geometry>
+				<cylinder length="0.18" radius="0.036"/>
+			</geometry>
 		</collision>
 	</link>
@@ -86,8 +86,8 @@
 		</visual>
 		<collision>
+			<origin xyz = "0.0 0 0.039 " rpy = " ${pi/2} ${pi/2} ${pi/2}"/>
 		  	<geometry>
-		   		<mesh filename="file://$(find mycobot_description)/urdf/mesh/link3.dae"/>
-		  	</geometry>
-		  	<origin xyz = "0.0 0 0.039 " rpy = " ${pi/2} ${pi/2} ${pi/2}"/>
+		   		<cylinder length="0.14" radius="0.0305"/>
+		  	</geometry>
 		</collision>
 	</link>
@@ -108,8 +108,8 @@
 		</visual>
 		<collision>
-			<geometry>
-				<mesh filename="file://$(find mycobot_description)/urdf/mesh/link4.dae"/>
-			</geometry>
 			<origin xyz = "0.0 -0.0024 -0.05 " rpy = "${pi/2} ${pi/2} 0 "/>
+			<geometry>
+				<cylinder length="0.083" radius="0.029"/>
+			</geometry>
 		</collision>
 	</link>
@@ -130,8 +130,8 @@
 		</visual>
 		<collision>
+		  	<origin xyz = "0.0 0 -0.05 " rpy = "0 0 ${-pi/2}"/>
 		   	<geometry>
-		   		<mesh filename="file://$(find mycobot_description)/urdf/mesh/link5.dae"/>
-		  	</geometry>
-		  	<origin xyz = "0.0 0 -0.05 " rpy = "0 0 ${-pi/2}"/>
+		   		<cylinder length="0.0849" radius="0.029"/>
+		  	</geometry>
 		</collision>
 	</link>
@@ -155,8 +155,8 @@
 		</visual>
 		<collision>
+		  	<origin xyz = "0.0 0.0 -0.022 " rpy = " ${pi/2} ${pi/2} 0"/>
 		   	<geometry>
-		   		<mesh filename="file://$(find mycobot_description)/urdf/mesh/link6.dae"/>
-		  	</geometry>
-		  	<origin xyz = "0.0 0.0 -0.022 " rpy = " ${pi/2} ${pi/2} 0"/>
+		   		<cylinder length="0.0225" radius="0.026"/>
+		  	</geometry>
 		</collision>
 	</link>
