Commit message: progress update
moveit2 integration wip

File: ros2/ros2-pkg/hos-resolve/src/mycobot_description/urdf/xacro/mycobot_320_pi_ros2control.urdf.xacro (robot description, xacro)
@@ -2,5 +2,5 @@
 <robot xmlns:xacro="http://wiki.ros.org/xacro" name="mycobot_320pi">
 	<link name="world"/>
-	<xacro:property name="effort" value="5.0"/> <!-- TODO: effort is 1000.00?? -->
+	<xacro:property name="effort" value="1000.0"/>
 	<xacro:property name="velocity" value="2.792527"/>
 	<link name="base">
@@ -26,5 +26,4 @@
 		</collision>
 	</link>
-	<!--Define the first link of the robotic arm. Each link represents a solid part of the robot.-->
 	<link name="link1">
 		<inertial>
@@ -49,5 +48,4 @@
 		</collision>
 	</link>
-	<!-- Define the second link of the robotic arm, and so on.-->
 	<link name="link2">
 		<inertial>
@@ -185,6 +183,4 @@
         <material>Gazebo/White</material>
     </gazebo>
-	<!-- ********** JOINTS ********** -->
-	<!-- Attach the robot base to the world frame with no initial offset or rotation. -->
 	<joint name="virtual_joint" type="fixed">
 		<parent link="world"/>
