Commit message: uploading working version

File: ros2/ros2-pkg/hos-resolve/src/mycobot_description/config/mycobot.urdf.xacro (robot description, xacro)
@@ -1,9 +1,9 @@
 <?xml version="1.0"?>
-<robot xmlns:xacro="http://www.ros.org/wiki/xacro" name="mycobot_320pi">
+<robot xmlns:xacro="http://www.ros.org/wiki/xacro" name="mycobot">
     <xacro:arg name="initial_positions_file" default="initial_positions.yaml" />
     <!-- Import firefighter urdf file -->
-    <xacro:include filename="$(find mycobot_description)/obj/original/mycobot_320_pi_moveit_2022.urdf" />
+    <xacro:include filename="$(find mycobot_description)/obj/urdf/mycobot_320_pi_moveit_2022_gz.urdf" />
     <!-- Import control_xacro -->
     <xacro:include filename="mycobot.ros2_control.xacro" />
-    <xacro:firefighter_ros2_control name="FakeSystem" initial_positions_file="$(arg initial_positions_file)"/>
+    <xacro:mycobot_ros2_control name="FakeSystem" initial_positions_file="$(arg initial_positions_file)"/>
 </robot>

File: ros2/ros2-pkg/hos-resolve/src/mycobot_description/obj/urdf/mycobot_320_pi_moveit_2022.urdf (robot description, URDF)
Before this commit: robot firefighter, 7 links, 6 joints
Links:
- link base: geometry collision cylinder length=0.102 radius=0.0725; visual mesh filename=package://mycobot_description/obj/mesh/base.dae
- link link1: geometry collision cylinder length=0.106 radius=0.043; visual mesh filename=package://mycobot_description/obj/mesh/link1.dae
- link link2: geometry collision cylinder length=0.18 radius=0.036; visual mesh filename=package://mycobot_description/obj/mesh/link2.dae
- link link4: geometry collision cylinder length=0.083 radius=0.029; visual mesh filename=package://mycobot_description/obj/mesh/link4.dae
- link link5: geometry collision cylinder length=0.0849 radius=0.029; visual mesh filename=package://mycobot_description/obj/mesh/link5.dae
- link link6: geometry collision cylinder length=0.0225 radius=0.026; visual mesh filename=package://mycobot_description/obj/mesh/link6.dae

File: ros2/ros2-pkg/hos-resolve/src/mycobot_description/obj/urdf/mycobot_320_pi_moveit_2022_gz.urdf (robot description, URDF)
Before this commit: robot firefighter, 7 links, 6 joints
Links:
- link base: geometry collision cylinder length=0.102 radius=0.0725; visual mesh filename=file://$(find mycobot_description)/obj/mesh/base.dae
- link link1: geometry collision cylinder length=0.106 radius=0.043; visual mesh filename=file://$(find mycobot_description)/obj/mesh/link1.dae
- link link2: geometry collision cylinder length=0.18 radius=0.036; visual mesh filename=file://$(find mycobot_description)/obj/mesh/link2.dae
- link link3: geometry collision cylinder length=0.14 radius=0.0305; visual mesh filename=file://$(find mycobot_description)/obj/mesh/link3.dae
- link link4: geometry collision cylinder length=0.083 radius=0.029; visual mesh filename=file://$(find mycobot_description)/obj/mesh/link4.dae
- link link5: geometry collision cylinder length=0.0849 radius=0.029; visual mesh filename=file://$(find mycobot_description)/obj/mesh/link5.dae
- link link6: geometry collision cylinder length=0.0225 radius=0.026; visual mesh filename=file://$(find mycobot_description)/obj/mesh/link6.dae
