Commit message: organize & release new hos ros

File: hos-resolve/src/mycobot_description/obj/urdf/new_mycobot_pro_320_pi_2022_moveit_gripper.urdf (robot description, URDF)
Before this commit: robot firefighter, 14 links, 13 joints
Links:
- link base: geometry collision cylinder length=0.102 radius=0.0725; visual mesh filename=package://mycobot_description/obj/mesh/base.dae
- link gripper_base: geometry collision mesh filename=package://mycobot_description/obj/mesh/gripper_base.dae; visual mesh filename=package://mycobot_description/obj/mesh/gripper_base.dae
- link gripper_left1: geometry collision mesh filename=package://mycobot_description/obj/mesh/gripper_left1.dae; visual mesh filename=package://mycobot_description/obj/mesh/gripper_left1.dae
- link gripper_left2: geometry collision mesh filename=package://mycobot_description/obj/mesh/gripper_left2.dae; visual mesh filename=package://mycobot_description/obj/mesh/gripper_left2.dae
- link gripper_left3: geometry collision mesh filename=package://mycobot_description/obj/mesh/gripper_left3.dae; visual mesh filename=package://mycobot_description/obj/mesh/gripper_left3.dae
- link gripper_right1: geometry collision mesh filename=package://mycobot_description/obj/mesh/gripper_right1.dae; visual mesh filename=package://mycobot_description/obj/mesh/gripper_right1.dae
- link gripper_right2: geometry collision mesh filename=package://mycobot_description/obj/mesh/gripper_right2.dae; visual mesh filename=package://mycobot_description/obj/mesh/gripper_right2.dae
- link gripper_right3: geometry collision mesh filename=package://mycobot_description/obj/mesh/gripper_right3.dae; visual mesh filename=package://mycobot_description/obj/mesh/gripper_right3.dae
- link link1: geometry collision cylinder length=0.106 radius=0.043; visual mesh filename=package://mycobot_description/obj/mesh/link1.dae
- link link2: geometry collision cylinder length=0.18 radius=0.036; visual mesh filename=package://mycobot_description/obj/mesh/link2.dae
- link link3: geometry collision cylinder length=0.14 radius=0.0305; visual mesh filename=package://mycobot_description/obj/mesh/link3.dae
- link link4: geometry collision cylinder length=0.083 radius=0.029; visual mesh filename=package://mycobot_description/obj/mesh/link4.dae
- link link5: geometry collision cylinder length=0.0849 radius=0.029; visual mesh filename=package://mycobot_description/obj/mesh/link5.dae
- link link6: geometry collision cylinder length=0.0225 radius=0.026; visual mesh filename=package://mycobot_description/obj/mesh/link6.dae
